File: WB/WB.kicad_pcb (KiCad board)
At the start: 2 copper layers, 140.3 x 89.7 mm, 47 parts, among them J1 Conn_01x04, J2 Conn_01x04, J3 Conn_01x04, J4 Conn_01x04, J5 Pump, J6 Actuator, J7 Actuator, J8 Screw_Terminal_01x02, M1 Fan, Q1 Q_NMOS_GDS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

Commit message: 回路図の修正
Parts:
- added C1: C, Capacitor_THT:C_Rect_L4.0mm_W2.5mm_P2.50mm, F.Cu at (167.3, 83.5)
- added C2: C, Capacitor_THT:C_Radial_D8.0mm_H11.5mm_P3.50mm, F.Cu at (184.0, 88.5)
- added C3: C, Capacitor_THT:C_Rect_L4.0mm_W2.5mm_P2.50mm, F.Cu at (188.0, 121.5)
- added C4: C, Capacitor_THT:C_Rect_L4.0mm_W2.5mm_P2.50mm, F.Cu at (186.6, 127.1)
- moved U2 3.69 mm to (176.5, 77.1)
- moved U3 1.15 mm to (174.5, 90.7)
Connections:
- Q7 pad 1: Net-(A4-Pad5) -> Net-(Q7-Pad1)
- U1 pad 1: Net-(A4-Pad8) -> Net-(U1-Pad1)
- U1 pad 2: Net-(A4-Pad7) -> Net-(U1-Pad2)
- U1 pad 9: Net-(A4-Pad6) -> Net-(U1-Pad9)
- U2 pad 11: Net-(A4-Pad11) -> Net-(U2-Pad11)
- U2 pad 12: Net-(A4-Pad10) -> Net-(U2-Pad12)
- U2 pad 14: Net-(A4-Pad9) -> Net-(U2-Pad14)
Routing:
- net Net-(Q7-Pad1): track 0.00 -> 183.6 mm
- net Net-(A4-Pad5): track 183.6 -> 0.00 mm
- net Net-(U1-Pad9): track 0.00 -> 34.9 mm
- net Net-(A4-Pad6): track 34.9 -> 0.00 mm
- net +24V: track 431.6 -> 460.1 mm
- net GND: track 477.1 -> 499.7 mm
- net Net-(U2-Pad11): track 0.00 -> 19.0 mm
- net Net-(U2-Pad12): track 0.00 -> 18.7 mm
- net Net-(A4-Pad11): track 17.0 -> 0.00 mm
- net Net-(A4-Pad10): track 16.9 -> 0.00 mm
- net Net-(U2-Pad14): track 0.00 -> 16.5 mm
- net Net-(A4-Pad9): track 14.8 -> 0.00 mm
- net VCC: track 297.7 -> 290.7 mm
- net Net-(Q5-Pad1): track 35.0 -> 40.5 mm
- net Net-(Q6-Pad1): track 56.6 -> 60.8 mm
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
Commit message: 回路周りのファイル
Routing:
- net GND: track 499.7 -> 469.4 mm
- net VCC: track 290.7 -> 287.5 mm
Changed lines of the file:
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@@
   (segment (start 199.5105 129.034) (end 203.71 129.034) (width 2) (layer "F.Cu") (net 2))
   (segment (start 184.3135 111.252) (end 193.197 120.1355) (width 2) (layer "F.Cu") (net 2))
-  (segment (start 126.238 137.795) (end 135.636 137.795) (width 2) (layer "F.Cu") (net 2))
-  (segment (start 125.857 105.0925) (end 127.852534 105.0925) (width 2) (layer "F.Cu") (net 2))
   (segment (start 181.173068 59.294) (end 186.240068 64.361) (width 2) (layer "F.Cu") (net 2))
-  (segment (start 125.857 137.414) (end 126.238 137.795) (width 2) (layer "F.Cu") (net 2))
   (segment (start 195.197 120.1355) (end 197.2245 120.1355) (width 2) (layer "F.Cu") (net 2))
   (segment (start 113.324 116.673) (end 113.157 116.84) (width 2) (layer "F.Cu") (net 2))
@@
   (segment (start 192.969 88.519) (end 195.197 86.291) (width 2) (layer "F.Cu") (net 2))
   (segment (start 197.2245 120.1355) (end 199.4705 122.3815) (width 2) (layer "F.Cu") (net 2))
-  (segment (start 136.044034 96.901) (end 140.081 96.901) (width 2) (layer "F.Cu") (net 2))
   (segment (start 194.7405 120.1355) (end 195.197 120.1355) (width 2) (layer "F.Cu") (net 2))
   (segment (start 160.259 112.918) (end 160.259 114.935) (width 2) (layer "F.Cu") (net 2))
@@
   (segment (start 135.636 137.795) (end 174.132875 137.795) (width 2) (layer "F.Cu") (net 2))
   (segment (start 176.53 59.294) (end 181.173068 59.294) (width 2) (layer "F.Cu") (net 2))
-  (segment (start 125.857 134.62) (end 125.857 137.414) (width 2) (layer "F.Cu") (net 2))
   (segment (start 157.321 91.821) (end 155.321 91.821) (width 2) (layer "F.Cu") (net 2))
   (segment (start 174.498 93.178) (end 174.498 90.034466) (width 2) (layer "F.Cu") (net 2))
@@
   (segment (start 125.857 134.62) (end 125.817 134.58) (width 2) (layer "F.Cu") (net 2))
   (segment (start 157.719 103.315) (end 158.831581 102.202419) (width 2) (layer "F.Cu") (net 2))
-  (segment (start 127.852534 105.0925) (end 136.044034 96.901) (width 2) (layer "F.Cu") (net 2))
   (segment (start 157.719 110.348) (end 157.719 107.315) (width 2) (layer "F.Cu") (net 2))
   (segment (start 172.959 112.939466) (end 174.646466 111.252) (width 2) (layer "F.Cu") (net 2))
@@
   (segment (start 113.157 116.84) (end 110.109 116.84) (width 2) (layer "B.Cu") (net 2))
   (segment (start 115.152534 132.08) (end 113.157 132.08) (width 2) (layer "B.Cu") (net 2))
-  (segment (start 116.967 81.28) (end 124.841 81.28) (width 2) (layer "F.Cu") (net 3))
-  (segment (start 143.764 105.542) (end 143.764 92.964) (width 2) (layer "F.Cu") (net 3))
-  (segment (start 116.967 96.901) (end 117.221 97.155) (width 2) (layer "F.Cu") (net 3))
   (segment (start 158.674466 53.594) (end 110.617 53.594) (width 2) (layer "F.Cu") (net 3))
-  (segment (start 116.967 81.28) (end 116.967 96.901) (width 2) (layer "F.Cu") (net 3))
+  (segment (start 143.764 92.964) (end 143.764 105.542) (width 2) (layer "F.Cu") (net 3))
   (segment (start 175.499 120.508) (end 176.906 121.915) (width 2) (layer "F.Cu") (net 3))
+  (segment (start 135.382 91.821) (end 142.621 91.821) (width 2) (layer "F.Cu") (net 3))
   (segment (start 181.356 121.915) (end 181.864 121.915) (width 2) (layer "F.Cu") (net 3))
-  (segment (start 117.221 91.694) (end 117.221 97.155) (width 2) (layer "F.Cu") (net 3))
-  (segment (start 116.278709 119.38) (end 113.157 119.38) (width 2) (layer "F.Cu") (net 3))
-  (segment (start 143.764 92.964) (end 142.621 91.821) (width 2) (layer "F.Cu") (net 3))
+  (segment (start 143.764 105.542) (end 141.356 107.95) (width 2) (layer "F.Cu") (net 3))
+  (segment (start 124.841 81.28) (end 123.952 81.28) (width 2) (layer "F.Cu") (net 3))
+  (segment (start 115.152534 60.325) (end 113.157 60.325) (width 2) (layer "F.Cu") (net 3))
   (segment (start 109.474 54.737) (end 109.474 60.102) (width 2) (layer "F.Cu") (net 3))
-  (segment (start 115.3795 89.8525) (end 117.221 91.694) (width 2) (layer "F.Cu") (net 3))
-  (segment (start 117.221 118.437709) (end 116.278709 119.38) (width 2) (layer "F.Cu") (net 3))
+  (segment (start 123.952 81.28) (end 117.221 88.011) (width 2) (layer "F.Cu") (net 3))
+  (segment (start 116.617 89.8525) (end 116.967 89.5025) (width 2) (layer "F.Cu") (net 3))
   (segment (start 168.91 61.834) (end 166.914466 61.834) (width 2) (layer "F.Cu") (net 3))
-  (segment (start 135.382 91.821) (end 140.081 91.821) (width 2) (layer "F.Cu") (net 3))
+  (segment (start 113.157 89.8525) (end 116.617 89.8525) (width 2) (layer "F.Cu") (net 3))
   (segment (start 176.906 121.915) (end 181.356 121.915) (width 2) (layer "F.Cu") (net 3))
+  (segment (start 117.221 119.316) (end 117.221 88.011) (width 2) (layer "F.Cu") (net 3))
   (segment (start 166.914466 61.834) (end 158.674466 53.594) (width 2) (layer "F.Cu") (net 3))
   (segment (start 175.499 114.935) (end 175.499 120.508) (width 2) (layer "F.Cu") (net 3))
-  (segment (start 141.356 107.95) (end 143.764 105.542) (width 2) (layer "F.Cu") (net 3))
-  (segment (start 142.621 91.821) (end 140.081 91.821) (width 2) (layer "F.Cu") (net 3))
-  (segment (start 116.967 62.139466) (end 116.967 81.28) (width 2) (layer "F.Cu") (net 3))
   (segment (start 181.356 121.915) (end 181.356 121.793) (width 2) (layer "F.Cu") (net 3))
   (segment (start 141.356 107.95) (end 144.8816 111.4756) (width 2) (layer "F.Cu") (net 3))
-  (segment (start 113.157 89.8525) (end 115.3795 89.8525) (width 2) (layer "F.Cu") (net 3))
   (segment (start 124.841 81.28) (end 135.382 91.821) (width 2) (layer "F.Cu") (net 3))
-  (segment (start 115.152534 60.325) (end 116.967 62.139466) (width 2) (layer "F.Cu") (net 3))
   (segment (start 109.697 60.325) (end 113.157 60.325) (width 2) (layer "F.Cu") (net 3))
-  (segment (start 113.157 60.325) (end 115.152534 60.325) (width 2) (layer "F.Cu") (net 3))
   (segment (start 109.474 60.102) (end 109.697 60.325) (width 2) (layer "F.Cu") (net 3))
+  (segment (start 117.221 88.011) (end 117.221 62.393466) (width 2) (layer "F.Cu") (net 3))
   (segment (start 144.8816 111.4756) (end 144.8816 121.915) (width 2) (layer "F.Cu") (net 3))
-  (segment (start 117.221 97.155) (end 117.221 118.437709) (width 2) (layer "F.Cu") (net 3))
+  (segment (start 117.221 62.393466) (end 115.152534 60.325) (width 2) (layer "F.Cu") (net 3))
   (segment (start 135.763 121.915) (end 181.356 121.915) (width 2) (layer "F.Cu") (net 3))
+  (segment (start 142.621 91.821) (end 143.764 92.964) (width 2) (layer "F.Cu") (net 3))
+  (segment (start 117.157 119.38) (end 117.221 119.316) (width 2) (layer "F.Cu") (net 3))
   (segment (start 110.617 53.594) (end 109.474 54.737) (width 2) (layer "F.Cu") (net 3))
+  (segment (start 113.157 119.38) (end 117.157 119.38) (width 2) (layer "F.Cu") (net 3))
   (segment (start 166.914466 77.074) (end 168.91 77.074) (width 2) (layer "B.Cu") (net 3))
   (segment (start 164.425 64.323466) (end 164.425 74.584534) (width 2) (layer "B.Cu") (net 3))
@@
   (segment (start 178.831 66.914) (end 179.832 65.913) (width 2) (layer "B.Cu") (net 37))
   (segment (start 181.892 59.281) (end 195.2035 59.281) (width 2) (layer "B.Cu") (net 37))
-  (segment (start 125.603 66.675) (end 125.603 64.135) (width 2) (layer "F.Cu") (net 44))
+  (segment (start 125.857 65.405) (end 125.857 62.865) (width 2) (layer "F.Cu") (net 44))
   (segment (start 110.577 121.88) (end 110.617 121.92) (width 2) (layer "F.Cu") (net 47))
   (segment (start 110.617 121.92) (end 113.157 121.92) (width 2) (layer "F.Cu") (net 47))
@@
   (segment (start 194.437 132.715) (end 193.675 133.477) (width 2) (layer "F.Cu") (net 78))
   (segment (start 196.469 132.715) (end 194.437 132.715) (width 2) (layer "F.Cu") (net 78))
+  (segment (start 129.54 73.877534) (end 129.54 65.532) (width 2) (layer "F.Cu") (net 79))
+  (segment (start 129.54 65.532) (end 132.247 62.825) (width 2) (layer "F.Cu") (net 79))
+  (segment (start 139.233 62.825) (end 140.2255 63.8175) (width 2) (layer "F.Cu") (net 79))
   (segment (start 132.247 62.825) (end 139.233 62.825) (width 2) (layer "F.Cu") (net 79))
-  (segment (start 139.233 62.825) (end 140.2255 63.8175) (width 2) (layer "F.Cu") (net 79))
-  (segment (start 127.889 75.565) (end 129.54 73.914) (width 2) (layer "F.Cu") (net 79))
-  (segment (start 129.54 73.914) (end 129.54 65.532) (width 2) (layer "F.Cu") (net 79))
-  (segment (start 125.857 75.565) (end 127.889 75.565) (width 2) (layer "F.Cu") (net 79))
-  (segment (start 129.54 65.532) (end 132.247 62.825) (width 2) (layer "F.Cu") (net 79))
+  (segment (start 125.857 75.565) (end 127.852534 75.565) (width 2) (layer "F.Cu") (net 79))
+  (segment (start 127.852534 75.565) (end 129.54 73.877534) (width 2) (layer "F.Cu") (net 79))
   (segment (start 125.857 60.325) (end 151.765 60.325) (width 2) (layer "F.Cu") (net 80))
   (segment (start 151.765 60.325) (end 155.2575 63.8175) (width 2) (layer "F.Cu") (net 80))
